Commit message: double pendulum appears correct

File: C_Iris_Examples/assets/double_pendulum_world.urdf (robot description, URDF)
Before this commit: robot double_pendulum, 3 links, 3 joints
Links:
- link link2: geometry collision box size=0.5 0.5 0.5; visual box size=0.1 0.1 1

Commit message: checkpoint

File: C_Iris_Examples/assets/double_pendulum_world.urdf (robot description, URDF)
Before this commit: robot double_pendulum, 3 links, 3 joints
Links:
- link fixed: geometry collision box size=1 1 10; visual box size=1 1 10
